Commit message: Enable Gazebo support

File: urdf/barista_robot_model.urdf (robot description, URDF)
Before this commit: robot example_robot, 11 links, 10 joints
Links:
- link back_caster: mass None -> 0.25; geometry collision sphere radius=0.020; visual sphere radius=0.020
- link chassis: mass None -> 12; geometry collision cylinder length=0.155 radius=0.178; visual mesh filename=package://barista_robot_description/meshes/chassis.dae scale=1 1 1
- link cup_holder: mass None -> 6; geometry collision cylinder length=0.090 radius=0.160; visual mesh filename=package://barista_robot_description/meshes/cup_holder.dae scale=1 1 1
- link front_caster: mass None -> 0.25; geometry collision sphere radius=0.020; visual sphere radius=0.020
- link left_wheel: mass None -> 0.25; geometry collision cylinder length=0.040 radius=0.020; visual cylinder length=0.040 radius=0.020
- link right_wheel: mass None -> 0.25; geometry collision cylinder length=0.040 radius=0.020; visual cylinder length=0.040 radius=0.020
- link rod_a: mass None -> 0.25; geometry collision cylinder length=0.22 radius=0.01; visual cylinder length=0.22 radius=0.01
- link rod_b: mass None -> 0.25; geometry collision cylinder length=0.22 radius=0.01; visual cylinder length=0.22 radius=0.01
- link rod_c: mass None -> 0.25; geometry collision cylinder length=0.22 radius=0.01; visual cylinder length=0.22 radius=0.01
- link rod_d: mass None -> 0.25; geometry collision cylinder length=0.22 radius=0.01; visual cylinder length=0.22 radius=0.01
Joints:
- joint chassis_to_back_caster: axis 0 1 0 -> (none); type continuous -> fixed
- joint chassis_to_front_caster: axis 0 1 0 -> (none); type continuous -> fixed
- joint chassis_to_left_wheel: limit (none) -> effort=10000 velocity=1000
- joint chassis_to_right_wheel: limit (none) -> effort=10000 velocity=1000

Commit message: Add laser sensor

File: urdf/barista_robot_model.urdf (robot description, URDF)
Before this commit: robot barista_robot, 11 links, 10 joints
Links:
- added link laser_frame
- added link laser_sensor, mass 0.160; collision box size=0.050 0.050 0.070; visual mesh filename=package://barista_robot_description/meshes/hokuyo.dae scale=1 1 1
Joints:
- added joint chassis_to_laser_sensor: type fixed, parent chassis, child laser_sensor, origin xyz=0.130 0 0.0775 rpy=0 0 0
- added joint laser_sensor_to_laser_frame: type fixed, parent laser_sensor, child laser_frame, origin xyz=0 0 0.060 rpy=0 0 0

Commit message: Fix laser scan position for URDF

File: urdf/barista_robot_model.urdf (robot description, URDF)
Before this commit: robot barista_robot, 13 links, 12 joints
Links:
- link base_link: mass None -> 0.0001
- link laser_frame: mass None -> 0.0001
