Commit message: Fix laser scan positions for XACRO

File: xacro/barista_robot_model.urdf.xacro (robot description, xacro)
@@ -39,5 +39,10 @@
     </material>
     <!-- Reference Frame-->
-    <link name="base_link"/>
+    <link name="base_link">
+        <inertial>
+            <mass value="0.0001"/>
+            <inertia ixx="0.0001" ixy="0.0" ixz="0.0" iyy="0.0001" iyz="0.0" izz="0.0001"/>
+        </inertial>
+    </link>
     <!-- Chassis -->
     <link name="chassis">
@@ -72,4 +77,7 @@
         <origin xyz="0 0 ${wheel_radius + chassis_length / 2}" rpy="0 0 0"/>
     </joint>
+    <gazebo reference="reference_to_chassis">
+        <preserveFixedJoint>true</preserveFixedJoint>
+    </gazebo>
     <!-- Left Wheel -->
     <xacro:wheel link_name="left_wheel" radius="${wheel_radius}" width="${wheel_width}" mass="${wheel_mass}"/>
@@ -126,4 +134,7 @@
         <origin xyz="${standoff_x_offset} ${standoff_y_offset} ${chassis_length / 2 + standoff_length / 2}" rpy="0 0 0"/>
     </joint>
+    <gazebo reference="chassis_to_rod_a">
+        <preserveFixedJoint>true</preserveFixedJoint>
+    </gazebo>
     <!-- Rod B -->
     <xacro:standoff link_name="rod_b" radius="${standoff_radius}" length="${standoff_length}" mass="${standoff_mass}"/>
@@ -134,4 +145,7 @@
         <origin xyz="${-standoff_x_offset} ${standoff_y_offset} ${chassis_length / 2 + standoff_length / 2}" rpy="0 0 0"/>
     </joint>
+    <gazebo reference="chassis_to_rod_b">
+        <preserveFixedJoint>true</preserveFixedJoint>
+    </gazebo>
     <!-- Rod C -->
     <xacro:standoff link_name="rod_c" radius="${standoff_radius}" length="${standoff_length}" mass="${standoff_mass}"/>
@@ -142,4 +156,7 @@
         <origin xyz="${standoff_x_offset} ${-standoff_y_offset} ${chassis_length / 2 + standoff_length / 2}" rpy="0 0 0"/>
     </joint>
+    <gazebo reference="chassis_to_rod_c">
+        <preserveFixedJoint>true</preserveFixedJoint>
+    </gazebo>
     <!-- Rod D -->
     <xacro:standoff link_name="rod_d" radius="${standoff_radius}" length="${standoff_length}" mass="${standoff_mass}"/>
@@ -150,4 +167,7 @@
         <origin xyz="${-standoff_x_offset} ${-standoff_y_offset} ${chassis_length / 2 + standoff_length / 2}" rpy="0 0 0"/>
     </joint>
+    <gazebo reference="chassis_to_rod_d">
+        <preserveFixedJoint>true</preserveFixedJoint>
+    </gazebo>
     <!-- Cup Holder -->
     <xacro:cup_holder_tray radius="${cup_holder_radius}" length="${cup_holder_length}" mass="${cup_holder_mass}"/>
@@ -158,4 +178,7 @@
         <origin xyz="0 0 ${chassis_length / 2 + standoff_length + cup_holder_length / 2}" rpy="0 0 0"/>
     </joint>
+    <gazebo reference="chassis_to_cup_holder">
+        <preserveFixedJoint>true</preserveFixedJoint>
+    </gazebo>
     <!-- Laser Sensor -->
     <xacro:laser_scanner include_laser="${include_laser}"/>
@@ -166,4 +189,7 @@
         <origin xyz="${chassis_radius * 65 / 89.0} 0 ${chassis_length / 2}" rpy="0 0 0"/>
     </joint>
+    <gazebo reference="chassis_to_laser_sensor">
+        <preserveFixedJoint>true</preserveFixedJoint>
+    </gazebo>
     <!-- Joint State Plugin -->
     <gazebo>

File: xacro/laser_scanner.xacro (robot description, xacro)
@@ -24,5 +24,10 @@
             </link>
             <!-- Laser Frame-->
-            <link name="laser_frame"/>
+            <link name="laser_frame">
+                <inertial>
+                    <mass value="0.0001"/>
+                    <inertia ixx="0.0001" ixy="0.0" ixz="0.0" iyy="0.0001" iyz="0.0" izz="0.0001"/>
+                </inertial>
+            </link>
             <!-- Laser Sensor - Laser Frame -->
             <joint name="laser_sensor_to_laser_frame" type="fixed">
@@ -31,4 +36,7 @@
                 <origin xyz="0 0 0.060" rpy="0 0 0"/>
             </joint>
+            <gazebo reference="laser_sensor_to_laser_frame">
+                <preserveFixedJoint>true</preserveFixedJoint>
+            </gazebo>
             <!-- Laser Sensor Plugin -->
             <gazebo reference="laser_frame">

Commit message: Implement second robot instance with red skin

File: xacro/barista_robot_model.urdf.xacro (robot description, xacro)
@@ -7,8 +7,11 @@
     <xacro:include filename="$(find barista_robot_description)/xacro/cup_holder_tray.xacro"/>
     <xacro:include filename="$(find barista_robot_description)/xacro/laser_scanner.xacro"/>
+    <!--- General Properties -->
+    <xacro:property name="robot_name" value="$(arg robot_name)"/>
     <!-- Chassis Properties -->
     <xacro:property name="chassis_radius" value="0.178"/>
     <xacro:property name="chassis_length" value="0.155"/>
     <xacro:property name="chassis_mass" value="12"/>
+    <xacro:property name="chassis_red" value="$(arg chassis_red)"/>
     <!-- Wheel Properties -->
     <xacro:property name="wheel_radius" value="0.0352"/>
@@ -50,5 +53,10 @@
             <origin rpy="0 0 0" xyz="0 0 0"/>
             <geometry>
-                <mesh filename="package://barista_robot_description/meshes/chassis.dae" scale="1 1 1"/>
+                <xacro:if value="${chassis_red}">
+                    <mesh filename="package://barista_robot_description/meshes/chassis_red.dae" scale="1 1 1"/>
+                </xacro:if>
+                <xacro:unless value="${chassis_red}">
+                    <mesh filename="package://barista_robot_description/meshes/chassis.dae" scale="1 1 1"/>
+                </xacro:unless>
             </geometry>
         </visual>
@@ -171,5 +179,5 @@
     </gazebo>
     <!-- Cup Holder -->
-    <xacro:cup_holder_tray radius="${cup_holder_radius}" length="${cup_holder_length}" mass="${cup_holder_mass}"/>
+    <xacro:cup_holder_tray radius="${cup_holder_radius}" length="${cup_holder_length}" mass="${cup_holder_mass}" chassis_red="${chassis_red}"/>
     <!-- Chassis - Cup Holder -->
     <joint name="chassis_to_cup_holder" type="fixed">
@@ -182,5 +190,5 @@
     </gazebo>
     <!-- Laser Sensor -->
-    <xacro:laser_scanner include_laser="${include_laser}"/>
+    <xacro:laser_scanner robot_name="${robot_name}" include_laser="${include_laser}"/>
     <!-- Chassis - Laser Sensor -->
     <joint name="chassis_to_laser_sensor" type="fixed">
@@ -196,4 +204,5 @@
         <plugin name="barista_bot_joint_state" filename="libgazebo_ros_joint_state_publisher.so">
             <ros>
+                <namespace>/${robot_name}</namespace>
                 <remapping>~/out:=joint_states</remapping>
             </ros>
@@ -206,4 +215,8 @@
     <gazebo>
         <plugin filename="libgazebo_ros_diff_drive.so" name="differential_drive_controller">
+            <ros>
+                <namespace>/${robot_name}</namespace>
+                <remapping>/cmd_vel:=cmd_vel</remapping>
+            </ros>
             <!-- wheels -->
             <left_joint>chassis_to_left_wheel</left_joint>

File: xacro/cup_holder_tray.xacro (robot description, xacro)
@@ -1,10 +1,15 @@
 <?xml version="1.0"?>
 <robot xmlns:xacro="http://www.ros.org/wiki/xacro">
-    <xacro:macro name="cup_holder_tray" params="radius length mass">
+    <xacro:macro name="cup_holder_tray" params="radius length mass chassis_red:=false">
         <link name="cup_holder">
             <visual>
                 <origin rpy="0 0 0" xyz="0 0 0"/>
                 <geometry>
-                    <mesh filename="package://barista_robot_description/meshes/cup_holder.dae" scale="1 1 1"/>
+                    <xacro:if value="${chassis_red}">
+                        <mesh filename="package://barista_robot_description/meshes/cup_holder_red.dae" scale="1 1 1"/>
+                    </xacro:if>
+                    <xacro:unless value="${chassis_red}">
+                        <mesh filename="package://barista_robot_description/meshes/cup_holder.dae" scale="1 1 1"/>
+                    </xacro:unless>
                 </geometry>
             </visual>

File: xacro/laser_scanner.xacro (robot description, xacro)
@@ -1,5 +1,5 @@
 <?xml version="1.0"?>
 <robot xmlns:xacro="http://www.ros.org/wiki/xacro">
-    <xacro:macro name="laser_scanner" params="include_laser:=true">
+    <xacro:macro name="laser_scanner" params="robot_name include_laser:=true">
         <xacro:if value="${include_laser}">
             <!-- Laser Sensor -->
@@ -58,8 +58,9 @@
                     </ray>
                     <always_on>true</always_on>
-                    <visualize>true</visualize>
+                    <visualize>false</visualize>
                     <update_rate>100.0</update_rate>
-                    <plugin name="laser" filename="libgazebo_ros_ray_sensor.so">
+                    <plugin name="${robot_name}_laser" filename="libgazebo_ros_ray_sensor.so">
                         <ros>
+                            <namespace>/${robot_name}</namespace>
                             <remapping>~/out:=scan</remapping>
                         </ros>

Commit message: Implement common frame 'world' for both robots

File: xacro/barista_robot_model.urdf.xacro (robot description, xacro)
@@ -94,5 +94,5 @@
         <parent link="chassis"/>
         <child link="left_wheel"/>
-        <origin xyz="0 ${-wheel_separation / 2} ${-chassis_length / 2}" rpy="0 0 0"/>
+        <origin xyz="0 ${wheel_separation / 2} ${-chassis_length / 2}" rpy="0 0 0"/>
         <axis xyz="0 1 0"/>
         <limit effort="10000" velocity="1000" />
@@ -105,5 +105,5 @@
         <parent link="chassis"/>
         <child link="right_wheel"/>
-        <origin xyz="0 ${wheel_separation / 2} ${-chassis_length / 2}" rpy="0 0 0"/>
+        <origin xyz="0 ${-wheel_separation / 2} ${-chassis_length / 2}" rpy="0 0 0"/>
         <axis xyz="0 1 0"/>
         <limit effort="10000" velocity="1000" />
@@ -231,6 +231,6 @@
             <publish_odom>true</publish_odom>
             <publish_odom_tf>true</publish_odom_tf>
-            <odometry_frame>odom</odometry_frame>
-            <robot_base_frame>base_link</robot_base_frame>
+            <odometry_frame>${robot_name}/odom</odometry_frame>
+            <robot_base_frame>${robot_name}/base_link</robot_base_frame>
         </plugin>
     </gazebo>

File: xacro/laser_scanner.xacro (robot description, xacro)
@@ -41,5 +41,5 @@
             <!-- Laser Sensor Plugin -->
             <gazebo reference="laser_frame">
-                <sensor name="sensor_ray" type="ray">
+                <sensor name="${robot_name}_sensor_ray" type="ray">
                     <pose>0 0 0 0 0 0</pose>
                     <ray>
@@ -59,5 +59,5 @@
                     <always_on>true</always_on>
                     <visualize>false</visualize>
-                    <update_rate>100.0</update_rate>
+                    <update_rate>10.0</update_rate>
                     <plugin name="${robot_name}_laser" filename="libgazebo_ros_ray_sensor.so">
                         <ros>
@@ -65,4 +65,5 @@
                             <remapping>~/out:=scan</remapping>
                         </ros>
+                        <frame_name>${robot_name}/laser_frame</frame_name>
                         <output_type>sensor_msgs/LaserScan</output_type>
                     </plugin>
